File: delay_line_lumped_element.kicad_sch (KiCad schematic)
At the start: 13 parts, among them J1 Conn_Coaxial, J2 Conn_Coaxial

Commit message: Working on circuit in spice
Parts:
- added R1, R2: 50R, symbol Device:R_US
Connections:
- net GND: now also C1.2, C2.2, C3.2, C4.2, C5.2, C6.2, R2.2
- net sig_in: now also R1.1; no longer C1.1, L1.1
- net sig_out: now also R2.1
- new net: C1.1, L1.1, R1.2
Changed lines of the file:
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@@
     (company "HugonLabs")
   )
-  (junction (at 87.63 97.79) (diameter 0) (color 0 0 0 0)
-  )
   (junction (at 184.15 97.79) (diameter 0) (color 0 0 0 0)
   )
@@
   (junction (at 146.05 97.79) (diameter 0) (color 0 0 0 0)
   )
+  (junction (at 194.31 97.79) (diameter 0) (color 0 0 0 0)
+  )
   (wire (pts (xy 125.73 97.79) (xy 125.73 101.6))
     (stroke (width 0) (type default) (color 0 0 0 0))
@@
     (stroke (width 0) (type default) (color 0 0 0 0))
   )
+  (wire (pts (xy 194.31 97.79) (xy 195.58 97.79))
+    (stroke (width 0) (type default) (color 0 0 0 0))
+  )
   (wire (pts (xy 140.97 97.79) (xy 146.05 97.79))
     (stroke (width 0) (type default) (color 0 0 0 0))
@@
     (stroke (width 0) (type default) (color 0 0 0 0))
   )
-  (wire (pts (xy 184.15 97.79) (xy 195.58 97.79))
+  (wire (pts (xy 184.15 97.79) (xy 194.31 97.79))
     (stroke (width 0) (type default) (color 0 0 0 0))
   )
@@
     (stroke (width 0) (type default) (color 0 0 0 0))
   )
-  (wire (pts (xy 66.04 97.79) (xy 87.63 97.79))
+  (wire (pts (xy 66.04 97.79) (xy 80.01 97.79))
     (stroke (width 0) (type default) (color 0 0 0 0))
   )
@@
     (stroke (width 0) (type default) (color 0 0 0 0))
   )
+  (wire (pts (xy 194.31 110.49) (xy 195.58 110.49))
+    (stroke (width 0) (type default) (color 0 0 0 0))
+  )
   (wire (pts (xy 160.02 97.79) (xy 165.1 97.79))
+    (stroke (width 0) (type default) (color 0 0 0 0))
+  )
+  (wire (pts (xy 194.31 97.79) (xy 194.31 110.49))
     (stroke (width 0) (type default) (color 0 0 0 0))
   )
@@
     (pin "2")
   )
+  (symbol (lib_id "Device:R_US") (at 195.58 114.3 0) (unit 1)
+    (in_bom yes) (on_board yes) (fields_autoplaced)
+    (property "Reference" "R2" (id 0) (at 198.12 113.0299 0)
+      (effects (font (size 1.27 1.27)) (justify left))
+    )
+    (property "Value" "50R" (id 1) (at 198.12 115.5699 0)
+      (effects (font (size 1.27 1.27)) (justify left))
+    )
+    (property "Footprint" "" (id 2) (at 196.596 114.554 90)
+      (effects (font (size 1.27 1.27)) hide)
+    )
+    (property "Datasheet" "~" (id 3) (at 195.58 114.3 0)
+      (effects (font (size 1.27 1.27)) hide)
+    )
+    (pin "1")
+    (pin "2")
+  )
   (symbol (lib_id "Device:C") (at 87.63 105.41 0) (unit 1)
     (in_bom yes) (on_board yes) (fields_autoplaced)
@@
     (pin "1")
     (pin "2")
+  )
+  (symbol (lib_id "power:GND") (at 165.1 109.22 0) (unit 1)
+    (in_bom yes) (on_board yes) (fields_autoplaced)
+    (property "Reference" "#PWR06" (id 0) (at 165.1 115.57 0)
+      (effects (font (size 1.27 1.27)) hide)
+    )
+    (property "Value" "GND" (id 1) (at 165.1 114.3 0))
+    (property "Footprint" "" (id 2) (at 165.1 109.22 0)
+      (effects (font (size 1.27 1.27)) hide)
+    )
+    (property "Datasheet" "" (id 3) (at 165.1 109.22 0)
+      (effects (font (size 1.27 1.27)) hide)
+    )
+    (pin "1")
   )
   (symbol (lib_id "power:GND") (at 60.96 102.87 0) (unit 1)
@@
     )
     (property "Datasheet" "" (id 3) (at 60.96 102.87 0)
+      (effects (font (size 1.27 1.27)) hide)
+    )
+    (pin "1")
+  )
+  (symbol (lib_id "power:GND") (at 195.58 118.11 0) (unit 1)
+    (in_bom yes) (on_board yes) (fields_autoplaced)
+    (property "Reference" "#PWR08" (id 0) (at 195.58 124.46 0)
+      (effects (font (size 1.27 1.27)) hide)
+    )
+    (property "Value" "GND" (id 1) (at 195.58 123.19 0))
+    (property "Footprint" "" (id 2) (at 195.58 118.11 0)
+      (effects (font (size 1.27 1.27)) hide)
+    )
+    (property "Datasheet" "" (id 3) (at 195.58 118.11 0)
       (effects (font (size 1.27 1.27)) hide)
     )
@@
     (pin "2")
   )
+  (symbol (lib_id "power:GND") (at 106.68 109.22 0) (unit 1)
+    (in_bom yes) (on_board yes) (fields_autoplaced)
+    (property "Reference" "#PWR03" (id 0) (at 106.68 115.57 0)
+      (effects (font (size 1.27 1.27)) hide)
+    )
+    (property "Value" "GND" (id 1) (at 106.68 114.3 0))
+    (property "Footprint" "" (id 2) (at 106.68 109.22 0)
+      (effects (font (size 1.27 1.27)) hide)
+    )
+    (property "Datasheet" "" (id 3) (at 106.68 109.22 0)
+      (effects (font (size 1.27 1.27)) hide)
+    )
+    (pin "1")
+  )
   (symbol (lib_id "Device:L_Trim") (at 97.79 97.79 90) (unit 1)
     (in_bom yes) (on_board yes) (fields_autoplaced)
@@
     (pin "2")
   )
+  (symbol (lib_id "power:GND") (at 146.05 109.22 0) (unit 1)
+    (in_bom yes) (on_board yes) (fields_autoplaced)
+    (property "Reference" "#PWR05" (id 0) (at 146.05 115.57 0)
+      (effects (font (size 1.27 1.27)) hide)
+    )
+    (property "Value" "GND" (id 1) (at 146.05 114.3 0))
+    (property "Footprint" "" (id 2) (at 146.05 109.22 0)
+      (effects (font (size 1.27 1.27)) hide)
+    )
+    (property "Datasheet" "" (id 3) (at 146.05 109.22 0)
+      (effects (font (size 1.27 1.27)) hide)
+    )
+    (pin "1")
+  )
+  (symbol (lib_id "power:GND") (at 87.63 109.22 0) (unit 1)
+    (in_bom yes) (on_board yes) (fields_autoplaced)
+    (property "Reference" "#PWR02" (id 0) (at 87.63 115.57 0)
+      (effects (font (size 1.27 1.27)) hide)
+    )
+    (property "Value" "GND" (id 1) (at 87.63 114.3 0))
+    (property "Footprint" "" (id 2) (at 87.63 109.22 0)
+      (effects (font (size 1.27 1.27)) hide)
+    )
+    (property "Datasheet" "" (id 3) (at 87.63 109.22 0)
+      (effects (font (size 1.27 1.27)) hide)
+    )
+    (pin "1")
+  )
   (symbol (lib_id "Device:C") (at 146.05 105.41 0) (unit 1)
     (in_bom yes) (on_board yes) (fields_autoplaced)
@@
     (pin "1")
     (pin "2")
+  )
+  (symbol (lib_id "power:GND") (at 125.73 109.22 0) (unit 1)
+    (in_bom yes) (on_board yes) (fields_autoplaced)
+    (property "Reference" "#PWR04" (id 0) (at 125.73 115.57 0)
+      (effects (font (size 1.27 1.27)) hide)
+    )
+    (property "Value" "GND" (id 1) (at 125.73 114.3 0))
+    (property "Footprint" "" (id 2) (at 125.73 109.22 0)
+      (effects (font (size 1.27 1.27)) hide)
+    )
+    (property "Datasheet" "" (id 3) (at 125.73 109.22 0)
+      (effects (font (size 1.27 1.27)) hide)
+    )
+    (pin "1")
   )
   (symbol (lib_id "Connector:Conn_Coaxial") (at 60.96 97.79 0) (mirror y) (unit 1)
@@
     (pin "2")
   )
+  (symbol (lib_id "Device:R_US") (at 83.82 97.79 90) (unit 1)
+    (in_bom yes) (on_board yes) (fields_autoplaced)
+    (property "Reference" "R1" (id 0) (at 83.82 91.44 90))
+    (property "Value" "50R" (id 1) (at 83.82 93.98 90))
+    (property "Footprint" "" (id 2) (at 84.074 96.774 90)
+      (effects (font (size 1.27 1.27)) hide)
+    )
+    (property "Datasheet" "~" (id 3) (at 83.82 97.79 0)
+      (effects (font (size 1.27 1.27)) hide)
+    )
+    (pin "1")
+    (pin "2")
+  )
   (symbol (lib_id "power:GND") (at 200.66 100.33 0) (unit 1)
     (in_bom yes) (on_board yes) (fields_autoplaced)
-    (property "Reference" "#PWR02" (id 0) (at 200.66 106.68 0)
+    (property "Reference" "#PWR09" (id 0) (at 200.66 106.68 0)
       (effects (font (size 1.27 1.27)) hide)
     )
@@
     (pin "2")
   )
+  (symbol (lib_id "power:GND") (at 184.15 109.22 0) (unit 1)
+    (in_bom yes) (on_board yes) (fields_autoplaced)
+    (property "Reference" "#PWR07" (id 0) (at 184.15 115.57 0)
+      (effects (font (size 1.27 1.27)) hide)
+    )
+    (property "Value" "GND" (id 1) (at 184.15 114.3 0))
+    (property "Footprint" "" (id 2) (at 184.15 109.22 0)
+      (effects (font (size 1.27 1.27)) hide)
+    )
+    (property "Datasheet" "" (id 3) (at 184.15 109.22 0)
+      (effects (font (size 1.27 1.27)) hide)
+    )
+    (pin "1")
+  )
   (sheet_instances
     (path "/" (page "1"))
@@
       (reference "#PWR01") (unit 1) (value "GND") (footprint "")
     )
+    (path "/a65f4b08-ed17-4666-991e-102dbdbbb7ae"
+      (reference "#PWR02") (unit 1) (value "GND") (footprint "")
+    )
+    (path "/878c26d9-541e-4419-bfd9-495c7a099ac8"
+      (reference "#PWR03") (unit 1) (value "GND") (footprint "")
+    )
+    (path "/b4c981d3-33ad-4e3f-9cc0-0d593dfc06d9"
+      (reference "#PWR04") (unit 1) (value "GND") (footprint "")
+    )
+    (path "/95d8fdba-9829-48e8-8982-c38e02f78daf"
+      (reference "#PWR05") (unit 1) (value "GND") (footprint "")
+    )
+    (path "/6cedd722-1c91-4397-afa3-9c519f3265bd"
+      (reference "#PWR06") (unit 1) (value "GND") (footprint "")
+    )
+    (path "/fb20d7ad-617d-4b74-881a-fe167019ffa5"
+      (reference "#PWR07") (unit 1) (value "GND") (footprint "")
+    )
+    (path "/70ce59f9-e01c-4644-9298-11231313de3c"
+      (reference "#PWR08") (unit 1) (value "GND") (footprint "")
+    )
     (path "/f533bc4d-bd37-44a6-9486-0f0e7c9ed863"
-      (reference "#PWR02") (unit 1) (value "GND") (footprint "")
+      (reference "#PWR09") (unit 1) (value "GND") (footprint "")
     )
     (path "/6a0afaff-db1b-4e7f-91b7-1b9b68c64d60"
@@
       (reference "L5") (unit 1) (value "200n") (footprint "")
     )
-  )
+    (path "/dd5901c9-59a3-400c-af0f-32232f8eef54"
+      (reference "R1") (unit 1) (value "50R") (footprint "")
+    )
+    (path "/37b85a78-2b96-45f1-9436-17f2c308c9bc"
+      (reference "R2") (unit 1) (value "50R") (footprint "")
+    )
+  )
